File: cpu/cpu.kicad_pcb (KiCad board)
At the start: 4 copper layers, 102.4 x 40.3 mm, 44 parts, among them J2 Conn_01x08, Q1 AO3401A, Q2 RU1J002YN, Q3 RU1J002YN, U1 ICE40HX1K-VQ100_RV4028, U2 W25Q80DVSS, U3 AP2112K-1.2

Commit message: Improve power.  Start work on IO module
Parts:
- removed Q1: AO3401A, Package_TO_SOT_SMD:SOT-23
- removed Q2: RU1J002YN, Package_TO_SOT_SMD:SOT-323_SC-70
- removed R8: 39k, Resistor_SMD:R_0603_1608Metric
- removed R9: 3k3, Resistor_SMD:R_0603_1608Metric
- removed TP2: Test, TestPoint:TestPoint_Pad_1.5x1.5mm
- TP3: moved to F.Cu
- moved TP3 7.11 mm to (163.8, 102.2), turned to 0 degrees
- moved D1 1.71 mm to (160.0, 98.4)
- moved TP1 1.71 mm to (158.6, 95.6)
- moved C5 0.07 mm to (122.5, 109.6)
Connections:
- C11 pad 2: VCCIO -> +3V3
- C12 pad 2: VCCIO -> +3V3
- C13 pad 2: VCCIO -> +3V3
- C14 pad 2: VCCIO -> +3V3
- C15 pad 2: VCCIO -> +3V3
- C16 pad 2: VCCIO -> +3V3
- C17 pad 2: VCCIO -> +3V3
- C18 pad 2: VCCIO -> +3V3
- C19 pad 2: VCCIO -> +3V3
- C3 pad 1: +3V3 -> +5V
- C5 pad 1: VCCIO -> +3V3
- D1 pad 2: VCCIO -> +3V3
- J1 pad 78: unconnected-(J1-+5V-Pad78) -> +5V
- R10 pad 1: VCCIO -> +3V3
- R11 pad 1: VCCIO -> +3V3
- R3 pad 1: VCCIO -> +3V3
- R4 pad 1: VCCIO -> +3V3
- R5 pad 1: VCCIO -> +3V3
- R6 pad 1: VCCIO -> +3V3
- U1 pad 14: VCCIO -> +3V3
- U1 pad 22: VCCIO -> +3V3
- U1 pad 31: VCCIO -> +3V3
- U1 pad 38: VCCIO -> +3V3
- U1 pad 50: VCCIO -> +3V3
- U1 pad 58: VCCIO -> +3V3
- U1 pad 6: VCCIO -> +3V3
- U1 pad 67: VCCIO -> +3V3
- U1 pad 72: VCCIO -> +3V3
- U1 pad 88: VCCIO -> +3V3
- U1 pad 92: VCCIO -> +3V3
- U3 pad 1: +3V3 -> +5V
- U3 pad 3: +3V3 -> +5V
Routing:
- net VCCIO: track 50.2 -> 0.00 mm, vias 21 -> 0
- net +3V3: track 11.1 -> 60.9 mm, vias 0 -> 16
- net Net-(Q1-G): track 6.82 -> 0.00 mm
- net GND: track 52.7 -> 47.7 mm, vias 44 -> 43
- net Net-(Q2-D): track 2.19 -> 0.00 mm
- net +5V: track 0.00 -> 2.06 mm
- net Net-(D1-K): track 32.2 -> 30.5 mm
- added copper zone on B.Cu, net +3V3
- added copper zone on In1.Cu, net +3V3
- added copper zone on In2.Cu, net +3V3
- added copper zone on F.Cu, net +5V
- added copper zone on In2.Cu, net GND
- removed copper zone on F.Cu, net VCCIO
- removed copper zone on In2.Cu, net VCCIO
Other:
- board text added: "! Not 5V Compatible !"
- board text removed: "3v3"
