File: io/io.kicad_sch (KiCad schematic)
At the start: 43 parts, among them J2 Conn_01x03, J3 QwST, J4 SM03B-SRSS-TB, J5 QwST, J6 Conn_02x06_Odd_Even, SW1 SW_Push, SW2 SW_Push, U1 RP2350_80QFN, U2 74HC32, U3 W25Q32JVS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

Commit message: Updates to io board
Parts:
- J1: footprint (none) -> RV4028:ModuleHeader_Single
- U2: value 74HC32 -> 74AHC32
- U3: footprint Package_SO:SOIC-8_5.23x5.23mm_P1.27mm -> Package_SO:SOIC-8_5.3x5.3mm_P1.27mm
Changed lines of the file:
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@@
 			)
 		)
-		(property "Footprint" "Package_SO:SOIC-8_5.23x5.23mm_P1.27mm"
+		(property "Footprint" "Package_SO:SOIC-8_5.3x5.3mm_P1.27mm"
 			(at 99.06 171.45 0)
 			(effects
@@
 			)
 		)
-		(property "Value" "74HC32"
+		(property "Value" "74AHC32"
 			(at 137.16 38.0999 0)
 			(effects
@@
 			)
 		)
-		(property "Value" "74HC32"
+		(property "Value" "74AHC32"
 			(at 82.55 21.59 0)
 			(effects
@@
 			)
 		)
-		(property "Footprint" ""
+		(property "Footprint" "RV4028:ModuleHeader_Single"
 			(at 26.67 123.19 0)
 			(effects
@@
 			)
 		)
-		(property "Value" "74HC32"
+		(property "Value" "74AHC32"
 			(at 82.55 36.83 0)
 			(effects
@@
 			)
 		)
-		(property "Value" "74HC32"
+		(property "Value" "74AHC32"
 			(at 101.6 24.13 0)
 			(effects
@@
 			)
 		)
-		(property "Value" "74HC32"
+		(property "Value" "74AHC32"
 			(at 82.55 77.47 0)
 			(effects

Commit message: IO module routed
Parts:
- added J7: Conn_01x03, Connector_PinSocket_2.54mm:PinSocket_1x03_P2.54mm_Vertical, symbol Connector_Generic:Conn_01x03
- added J8: Conn_01x01, Connector_PinHeader_2.54mm:PinHeader_1x01_P2.54mm_Vertical, symbol Connector_Generic:Conn_01x01
- added R5: 27, Resistor_SMD:R_0402_1005Metric, symbol Device:R
- J2: value Conn_01x03 -> Conn_02x03; footprint Connector_PinHeader_2.54mm:PinHeader_1x03_P2.54mm_Vertical -> Connector_PinHeader_2.54mm:PinHeader_2x03_P2.54mm_Vertical; symbol Connector_Generic:Conn_01x03 -> Connector_Generic:Conn_02x03_Odd_Even
- U1: footprint RP2350_80QFN_minimal:RP2350-QFN-80-1EP_10x10_P0.4mm_EP3.4x3.4mm_ThermalVias -> RV4028:RP2350-QFN-80-1EP_10x10_P0.4mm_EP3.4x3.4mm_ThermalVias
Connections:
- net +3V3: now also J7.3 (Pin_3)
- net +5V: now also J2.2 (Pin_2), J7.1 (Pin_1)
- net CLK: now also R5.1; no longer U1.19 (GPIO19)
- net GND: now also J2.5 (Pin_5), J2.6 (Pin_6), J7.2 (Pin_2); no longer J2.3 (Pin_3)
- net WS2812_DAT: now also J2.3 (Pin_3), J2.4 (Pin_4); no longer J2.2 (Pin_2)
- net ~{WAIT}: now also J8.1 (Pin_1)
- new net: R5.2, U1.19 (GPIO19)
- no-connect marks 7 -> 8
Other:
- moved on the sheet: C6, C7, C9, L1, R3, R4, R6, R7, R8, SW1, SW2, U1

Commit message: RAM module, many tweaks
Parts:
- D2: JLC (none) -> C42417498
- J1: JLC C3410 -> C2334
- J3, J5: JLC C160390 -> C160404
- J4: JLC (none) -> C160403
- J6: value Conn_02x06_Odd_Even -> Conn_02x08_Odd_Even; footprint Connector_PinHeader_2.54mm:PinHeader_2x06_P2.54mm_Vertical -> Connector_PinHeader_2.54mm:PinHeader_2x08_P2.54mm_Vertical; symbol Connector_Generic:Conn_02x06_Odd_Even -> Connector_Generic:Conn_02x08_Odd_Even
- L1: JLC (none) -> C42411119
- SW1, SW2: footprint Button_Switch_SMD:SW_Push_1P1T_NO_Vertical_Wuerth_434133025816 -> RV4028:SW-SMD_HX-TS-1101-C-W; JLC (none) -> C36498960
- U2: JLC (none) -> C132988
- Y1: JLC (none) -> C20625731
Connections:
- net +3V3: now also J6.1 (Pin_1), J6.15 (Pin_15), J6.2 (Pin_2); no longer J6.11 (Pin_11)
- net GND: now also J6.3 (Pin_3), J6.8 (Pin_8)
- net GPIO46_ADC6: now also J6.9 (Pin_9); no longer J6.5 (Pin_5)
- net GPIO47_ADC7: now also J6.7 (Pin_7); no longer J6.3 (Pin_3)
- net SPI_CLK: now also J6.14 (Pin_14); no longer J6.10 (Pin_10)
- net SPI_CS: now also J6.16 (Pin_16); no longer J6.12 (Pin_12)
- net SPI_CS1: now also J6.13 (Pin_13); no longer J6.9 (Pin_9)
- net SPI_CS2: now also J6.11 (Pin_11); no longer J6.7 (Pin_7)
- net SPI_RX: now also J6.12 (Pin_12); no longer J6.8 (Pin_8)
- net SPI_TX: now also J6.10 (Pin_10); no longer J6.6 (Pin_6)
- net UART0_RX: now also J6.6 (Pin_6); no longer J6.2 (Pin_2)
- net UART0_TX: now also J6.5 (Pin_5); no longer J6.1 (Pin_1)

Commit message: Revised module header
Parts:
- removed J1: ~, RV4028:ModuleHeader_Single, symbol RV4028:Single_Conn
- removed J7: Conn_01x03, Connector_PinSocket_2.54mm:PinSocket_1x03_P2.54mm_Vertical, symbol Connector_Generic:Conn_01x03
- removed J8: Conn_01x01, Connector_PinHeader_2.54mm:PinHeader_1x01_P2.54mm_Vertical, symbol Connector_Generic:Conn_01x01
- added J1: ~, RV4028:Module_2mm, symbol RV4028:Dual_Conn
- U2: value 74AHC32 -> 74LVC32; footprint Package_SO:SOIC-14_3.9x8.7mm_P1.27mm -> Package_SO:SSOP-14_5.3x6.2mm_P0.65mm
Connections:
- net +3V3: now also J1.18 (+3V3), J1.58 (+3V3)
- net +5V: now also J1.40 (+5V), J1.80 (+5V)
- net A0: now also J1.16 (A0)
- net A1: now also J1.15 (A1)
- net A2: now also J1.14 (A2)
- net A28: now also J1.3 (A28)
- net A29: now also J1.2 (A29)
- net A3: now also J1.13 (A3)
- net A30: now also J1.1 (A30)
- net A4: now also J1.12 (A4)
- net A5: now also J1.11 (A5)
- net A6: now also J1.10 (A6)
- net A7: now also J1.9 (A7)
- net CLK: now also J1.21 (CLK)
- net D0: now also J1.27 (D0)
- net D1: now also J1.28 (D1)
- net D2: now also J1.29 (D2)
- net D3: now also J1.30 (D3)
- net D4: now also J1.31 (D4)
- net D5: now also J1.32 (D5)
- net D6: now also J1.33 (D6)
- net D7: now also J1.34 (D7)
- net GND: now also J1.17 (GND), J1.39 (GND), J1.57 (GND), J1.60 (GND), J1.61 (GND), J1.66 (GND), J1.79 (GND)
- net UART1_RX: now also J1.36 (RX)
- net UART1_TX: now also J1.35 (TX)
- net USB_D+: now also J1.37 (USB_DP)
- net USB_D-: now also J1.38 (USB_DN)
- net ~{A31}: now also J1.26 (~{A31})
- net ~{INT}: now also J1.22 (~{INT})
- net ~{RD}: now also J1.25 (~{RD})
- net ~{REQ}: now also J1.23 (~{REQ})
- net ~{RESET}: now also J1.20 (~{RESET})
- net ~{WAIT}: now also J1.65 (~{WAIT})
- net ~{WR}: now also J1.24 (~{WR})
- no-connect marks 8 -> 39
Other:
- moved on the sheet: C19, U2A, U2B, U2C, U2D, U2E

Commit message: IO module 2mm headers
Parts:
- added R10, R11, R12, R9: 10k, Resistor_SMD:R_0402_1005Metric, symbol Device:R
Connections:
- net +3V3: now also R10.2, R11.2, R12.2, R9.2
- net I2C0_SCL: now also R10.1
- net I2C0_SDA: now also R9.1
- net I2C1_SCL: now also R11.1
- net I2C1_SDA: now also R12.1
- net USB_D+: now also J1.78 (USB_DP); no longer J1.37 (USB_DP)
- net USB_D-: now also J1.77 (USB_DN); no longer J1.38 (USB_DN)
- net WS2812_DAT: no longer J2.3 (Pin_3)
- new net S2: J1.38 (SPARE2), J2.3 (Pin_3)
- no-connect marks 39 -> 38
Other:
- moved on the sheet: J2, J5

Commit message: CPU and IO production fixes
Parts:
- J1: JLC C3410 -> C3407
- U1: JLC (none) -> C42415655
- U2: JLC C132988 -> C2867091
- U3: JLC (none) -> C179173
Changed lines of the file:
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@@
 			)
 		)
+		(property "JLC" "C179173"
+			(at 99.06 171.45 0)
+			(effects
+				(font
+					(size 1.27 1.27)
+				)
+				(hide yes)
+			)
+		)
 		(pin "1"
 		)
@@
 			)
 		)
-		(property "JLC" "C3410"
+		(property "JLC" "C3407"
 			(at 40.64 123.19 0)
 			(effects
@@
 			)
 		)
-		(property "JLC" "C132988"
+		(property "JLC" "C2867091"
 			(at 140.97 36.83 0)
 			(effects
@@
 			)
 		)
-		(property "JLC" "C132988"
+		(property "JLC" "C2867091"
 			(at 93.98 27.94 0)
 			(effects
@@
 			)
 		)
-		(property "JLC" "C132988"
+		(property "JLC" "C2867091"
 			(at 93.98 43.18 0)
 			(effects
@@
 			)
 		)
+		(property "JLC" "C42415655"
+			(at 213.36 120.65 0)
+			(effects
+				(font
+					(size 1.27 1.27)
+				)
+				(hide yes)
+			)
+		)
 		(pin "1"
 		)
@@
 			)
 		)
-		(property "JLC" "C132988"
+		(property "JLC" "C2867091"
 			(at 113.03 30.48 0)
 			(effects
@@
 			)
 		)
-		(property "JLC" "C132988"
+		(property "JLC" "C2867091"
 			(at 95.25 83.82 0)
 			(effects

Commit message: Add backplane
Parts:
- R5: value 27 -> 33
Changed lines of the file:
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@@
 			)
 		)
-		(property "Value" "27"
+		(property "Value" "33"
 			(at 273.05 132.9436 90)
 			(effects

Commit message: PDFs of schematics, readme updates
Other:
- company: (none) -> Team Rebellion
- title: (none) -> RV4028 IO Module
Changed lines of the file:
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@@
 	(generator_version "9.0")
 	(paper "A3")
+	(title_block
+		(title "RV4028 IO Module")
+		(date "2026-01-22")
+		(rev "v0.1")
+		(company "Team Rebellion")
+	)
 	(circle
 		(center 148.59 81.915)
