File: io/io.kicad_sch (KiCad schematic)
At the start: 48 parts, among them J2 Conn_02x03, J3 QwST, J4 SM03B-SRSS-TB, J5 QwST, J6 Conn_02x08_Odd_Even, SW1 SW_Push, SW2 SW_Push, U1 RP2350_80QFN, U2 74LVC32, U3 W25Q32JVS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

Commit message: Review before first PCB order
Parts:
- J2: JLC (none) -> C5383104
- J6: JLC (none) -> C5383108
Changed lines of the file:
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@@
+			)
+		)
+		(property "JLC" "C5383108"
+			(at 300.99 224.79 0)
+			(effects
+				(font
+					(size 1.27 1.27)
+				)
+				(hide yes)
 			)
 		)
@@
 			(at 394.97 232.41 0)
 			(effects
+				(font
+					(size 1.27 1.27)
+				)
+				(hide yes)
+			)
+		)
+		(property "JLC" "C5383104"
+			(at 394.97 232.41 0)
+			(effects
