File: ram/ram.kicad_sch (KiCad schematic)
At the start: 7 parts, among them J2 Conn_01x03, U1 IS66WVE4M16EBLL-70BLI, U3 74LVC2G00

Commit message: Revised module header
Parts:
- removed U3: 74LVC2G00, Package_SO:VSSOP-8_2.3x2mm_P0.5mm, symbol 74xGxx:74LVC2G00
- added C5: 100n, Capacitor_SMD:C_0402_1005Metric, symbol Device:C
- added J3: Conn_01x03, Connector_PinHeader_2.54mm:PinHeader_1x03_P2.54mm_Vertical, symbol Connector_Generic:Conn_01x03
- added U2: 74LVC32, Package_SO:SSOP-14_5.3x6.2mm_P0.65mm, symbol 74xx:74LS32
- added U3: 74LVC2G04, Package_TO_SOT_SMD:SOT-363_SC-70-6, symbol 74xGxx:74LVC2G04
Connections:
- net +3V3: now also J1.18 (+3V3), J1.58 (+3V3), C5.1, U2.14 (VCC), U3.5 (VCC); no longer J1.40 (+3V3), J1.80 (+3V3)
- net A23: now also U3.1
- net GND: now also J1.60 (GND), J1.61 (GND), J1.66 (GND), C5.2, U2.7 (GND), U3.2 (GND)
- net ~{A23}: now also U3.6
- net ~{CE}: now also U2.8
- net at J2.2 (Pin_2): now also U2.2
- net ~{REQ}: now reaches J1.23 (~{REQ})
- net ~{REQ}: now also U2.5
- net A24: now reaches J1.48 (A24)
- net A24: now also J3.1 (Pin_1), U3.3
- net LO_ADDR renamed ~{LO_ADDR}
- net ~{LO_ADDR}: now also U2.4
- new net: U2.10, U2.6
- new net: J3.2 (Pin_2), U2.1
- new net: U2.3, U2.9
- new net ~{A24}: J3.3 (Pin_3), U3.4
- no-connect marks 30 -> 28
Other:
- moved on the sheet: J2

Commit message: RAM board attempt 2
Parts:
- J1: footprint RV4028:ModuleHeader -> RV4028:Module_2mm; JLC C3410 -> C3407
Changed lines of the file:
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@@
 			)
 		)
-		(property "Footprint" "RV4028:ModuleHeader"
+		(property "Footprint" "RV4028:Module_2mm"
 			(at 49.53 135.89 0)
 			(effects
@@
 			)
 		)
-		(property "JLC" "C3410"
+		(property "JLC" "C3407"
 			(at 49.53 135.89 0)
 			(effects

Commit message: PDFs of schematics, readme updates
Other:
- company: (none) -> Team Rebellion
- title: (none) -> RV4028 RAM Module
Changed lines of the file:
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@@
 	(generator_version "9.0")
 	(paper "A4")
+	(title_block
+		(title "RV4028 RAM Module")
+		(date "2026-01-22")
+		(rev "v0.1")
+		(company "Team Rebellion")
+	)
 	(junction
 		(at 91.44 181.61)

Commit message: Pull up on REQ
Parts:
- U1: JLC (none) -> C1350157
Changed lines of the file:
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@@
+			)
+		)
+		(property "JLC" "C1350157"
+			(at 187.96 88.9 0)
+			(effects
+				(font
+					(size 1.27 1.27)
+				)
+				(hide yes)
 			)
 		)

Commit message: Review before first PCB order
Parts:
- J2, J3: JLC (none) -> C49257
Changed lines of the file:
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@@
+			)
+		)
+		(property "JLC" "C49257"
+			(at 110.49 49.53 0)
+			(effects
+				(font
+					(size 1.27 1.27)
+				)
+				(hide yes)
 			)
 		)
@@
 			(at 110.49 38.1 0)
 			(effects
+				(font
+					(size 1.27 1.27)
+				)
+				(hide yes)
+			)
+		)
+		(property "JLC" "C49257"
+			(at 110.49 38.1 0)
+			(effects
